Commit message: feat: add wheel_radius param for rad/s to mm/s conversion
When wheel_radius is set (> 0), the hardware interface converts
rad/s from the controller to mm/s for the Arduino on write, and
mm to rad on read. Defaults to 0 (passthrough).

File: sar_description/urdf/ros2_control.urdf.xacro (robot description, xacro)
@@ -1,5 +1,5 @@
 <?xml version="1.0"?>
 <robot xmlns:xacro="http://wiki.ros.org/xacro">
-  <xacro:macro name="sar_ros2_control" params="mock:=false">
+  <xacro:macro name="sar_ros2_control" params="mock:=false wheel_radius:=0.0">
     <ros2_control name="sar_system" type="system">
       <hardware>
@@ -8,4 +8,5 @@
         <param name="baud_rate">115200</param>
         <param name="mock">${mock}</param>
+        <param name="wheel_radius">${wheel_radius}</param>
       </hardware>
       <joint name="fl_wheel_joint">

File: sar_description/urdf/sar_robot.urdf.xacro (robot description, xacro)
@@ -17,4 +17,4 @@
   <xacro:wheel side="rr" wheel_radius="${wheel_radius}"
     x="${-wheel_separation_x / 2}" y="${-wheel_separation_y / 2}" />
-  <xacro:sar_ros2_control mock="$(arg mock)" />
+  <xacro:sar_ros2_control mock="$(arg mock)" wheel_radius="${wheel_radius}" />
 </robot>

Commit message: It's working! (at least a bit)
- Added cheat sheet for some repetitive commands
- Improved launch file
- Calculate velocities in SarSystemHardware::read()

File: sar_description/urdf/ros2_control.urdf.xacro (robot description, xacro)
@@ -1,10 +1,10 @@
 <?xml version="1.0"?>
 <robot xmlns:xacro="http://wiki.ros.org/xacro">
-  <xacro:macro name="sar_ros2_control" params="mock:=false wheel_radius:=0.0">
-    <ros2_control name="sar_system" type="system">
+  <xacro:macro name="sar_ros2_control" params="mock:=false wheel_radius:=0.0 baud_rate:=115200 device:=/dev/ttyACM0">
+    <ros2_control name="SarSystemHardware" type="system">
       <hardware>
         <plugin>sar_control/SarSystemHardware</plugin>
-        <param name="device">/dev/ttyUSB0</param>
-        <param name="baud_rate">115200</param>
+        <param name="device">${device}</param>
+        <param name="baud_rate">${baud_rate}</param>
         <param name="mock">${mock}</param>
         <param name="wheel_radius">${wheel_radius}</param>

File: sar_description/urdf/sar_robot.urdf.xacro (robot description, xacro)
@@ -2,4 +2,6 @@
 <robot name="sar_robot" xmlns:xacro="http://wiki.ros.org/xacro">
   <xacro:arg name="mock" default="false" />
+  <xacro:arg name="baud_rate" default="115200" />
+  <xacro:arg name="device" default="/dev/ttyACM0" />
   <xacro:include filename="$(find sar_description)/urdf/body.urdf.xacro" />
   <xacro:include filename="$(find sar_description)/urdf/wheel.urdf.xacro" />
@@ -17,4 +19,4 @@
   <xacro:wheel side="rr" wheel_radius="${wheel_radius}"
     x="${-wheel_separation_x / 2}" y="${-wheel_separation_y / 2}" />
-  <xacro:sar_ros2_control mock="$(arg mock)" wheel_radius="${wheel_radius}" />
+  <xacro:sar_ros2_control mock="$(arg mock)" wheel_radius="${wheel_radius}" baud_rate="$(arg baud_rate)" device="$(arg device)" />
 </robot>

Commit message: Add rplidar

File: sar_description/urdf/ros2_control.urdf.xacro (robot description, xacro)
@@ -1,5 +1,5 @@
 <?xml version="1.0"?>
 <robot xmlns:xacro="http://wiki.ros.org/xacro">
-  <xacro:macro name="sar_ros2_control" params="mock:=false wheel_radius:=0.0">
+  <xacro:macro name="sar_ros2_control" params="mock:=false">
     <ros2_control name="sar_system" type="system">
       <hardware>
@@ -8,24 +8,19 @@
         <param name="baud_rate">115200</param>
         <param name="mock">${mock}</param>
-        <param name="wheel_radius">${wheel_radius}</param>
       </hardware>
       <joint name="fl_wheel_joint">
         <command_interface name="velocity" />
-        <state_interface name="position" />
         <state_interface name="velocity" />
       </joint>
       <joint name="fr_wheel_joint">
         <command_interface name="velocity" />
-        <state_interface name="position" />
         <state_interface name="velocity" />
       </joint>
       <joint name="rl_wheel_joint">
         <command_interface name="velocity" />
-        <state_interface name="position" />
         <state_interface name="velocity" />
       </joint>
       <joint name="rr_wheel_joint">
         <command_interface name="velocity" />
-        <state_interface name="position" />
         <state_interface name="velocity" />
       </joint>

File: sar_description/urdf/sar_robot.urdf.xacro (robot description, xacro)
@@ -5,7 +5,7 @@
   <xacro:include filename="$(find sar_description)/urdf/wheel.urdf.xacro" />
   <xacro:include filename="$(find sar_description)/urdf/ros2_control.urdf.xacro" />
-  <xacro:property name="wheel_radius" value="0.050" />
-  <xacro:property name="wheel_separation_x" value="0.170" />
-  <xacro:property name="wheel_separation_y" value="0.270" />
+  <xacro:property name="wheel_radius" value="0.03" />
+  <xacro:property name="wheel_separation_x" value="0.180" />
+  <xacro:property name="wheel_separation_y" value="0.178" />
   <xacro:body wheel_radius="${wheel_radius}" />
   <xacro:wheel side="fl" wheel_radius="${wheel_radius}"
@@ -17,4 +17,5 @@
   <xacro:wheel side="rr" wheel_radius="${wheel_radius}"
     x="${-wheel_separation_x / 2}" y="${-wheel_separation_y / 2}" />
-  <xacro:sar_ros2_control mock="$(arg mock)" wheel_radius="${wheel_radius}" />
+  <xacro:rplidar x="0.0" y="0.0" z="0.03"/>
+  <xacro:sar_ros2_control mock="$(arg mock)"/>
 </robot>

Commit message: General fixes for real hardware (#4)

File: sar_description/urdf/ros2_control.urdf.xacro (robot description, xacro)
@@ -1,10 +1,10 @@
 <?xml version="1.0"?>
 <robot xmlns:xacro="http://wiki.ros.org/xacro">
-  <xacro:macro name="sar_ros2_control" params="mock:=false">
+  <xacro:macro name="sar_ros2_control" params="mock:=false baud_rate:=115200 device:=/dev/ttyACM0">
     <ros2_control name="sar_system" type="system">
       <hardware>
         <plugin>sar_control/SarSystemHardware</plugin>
-        <param name="device">/dev/ttyUSB0</param>
-        <param name="baud_rate">115200</param>
+        <param name="device">${device}</param>
+        <param name="baud_rate">${baud_rate}</param>
         <param name="mock">${mock}</param>
       </hardware>

File: sar_description/urdf/sar_robot.urdf.xacro (robot description, xacro)
@@ -2,4 +2,6 @@
 <robot name="sar_robot" xmlns:xacro="http://wiki.ros.org/xacro">
   <xacro:arg name="mock" default="false" />
+  <xacro:arg name="baud_rate" default="115200" />
+  <xacro:arg name="device" default="/dev/ttyACM0" />
   <xacro:include filename="$(find sar_description)/urdf/body.urdf.xacro" />
   <xacro:include filename="$(find sar_description)/urdf/wheel.urdf.xacro" />
@@ -18,4 +20,4 @@
     x="${-wheel_separation_x / 2}" y="${-wheel_separation_y / 2}" />
   <xacro:rplidar x="0.0" y="0.0" z="0.03"/>
-  <xacro:sar_ros2_control mock="$(arg mock)"/>
+  <xacro:sar_ros2_control mock="$(arg mock)" baud_rate="$(arg baud_rate)" device="$(arg device)" />
 </robot>
