Commit message: Add rplidar to description

File: sar_description/urdf/body.urdf.xacro (robot description, xacro)
@@ -11,5 +11,5 @@
       <visual>
         <geometry>
-          <box size="0.240 0.220 0.060" />
+          <box size="0.240 0.178 0.060" />
         </geometry>
         <material name="dark_grey">
@@ -19,5 +19,5 @@
       <collision>
         <geometry>
-          <box size="0.240 0.220 0.060" />
+          <box size="0.240 0.178 0.060" />
         </geometry>
       </collision>

File: sar_description/urdf/ros2_control.urdf.xacro (robot description, xacro)
@@ -1,5 +1,5 @@
 <?xml version="1.0"?>
 <robot xmlns:xacro="http://wiki.ros.org/xacro">
-  <xacro:macro name="sar_ros2_control" params="mock:=false wheel_radius:=0.0 baud_rate:=115200 device:=/dev/ttyACM0">
+  <xacro:macro name="sar_ros2_control" params="mock:=false baud_rate:=115200 device:=/dev/ttyACM0">
     <ros2_control name="SarSystemHardware" type="system">
       <hardware>
@@ -8,24 +8,19 @@
         <param name="baud_rate">${baud_rate}</param>
         <param name="mock">${mock}</param>
-        <param name="wheel_radius">${wheel_radius}</param>
       </hardware>
       <joint name="fl_wheel_joint">
         <command_interface name="velocity" />
-        <state_interface name="position" />
         <state_interface name="velocity" />
       </joint>
       <joint name="fr_wheel_joint">
         <command_interface name="velocity" />
-        <state_interface name="position" />
         <state_interface name="velocity" />
       </joint>
       <joint name="rl_wheel_joint">
         <command_interface name="velocity" />
-        <state_interface name="position" />
         <state_interface name="velocity" />
       </joint>
       <joint name="rr_wheel_joint">
         <command_interface name="velocity" />
-        <state_interface name="position" />
         <state_interface name="velocity" />
       </joint>

File: sar_description/urdf/sar_robot.urdf.xacro (robot description, xacro)
@@ -7,7 +7,8 @@
   <xacro:include filename="$(find sar_description)/urdf/wheel.urdf.xacro" />
   <xacro:include filename="$(find sar_description)/urdf/ros2_control.urdf.xacro" />
-  <xacro:property name="wheel_radius" value="0.050" />
-  <xacro:property name="wheel_separation_x" value="0.170" />
-  <xacro:property name="wheel_separation_y" value="0.270" />
+  <xacro:include filename="$(find sar_description)/urdf/rplidar.urdf.xacro" />
+  <xacro:property name="wheel_radius" value="0.03" />
+  <xacro:property name="wheel_separation_x" value="0.180" />
+  <xacro:property name="wheel_separation_y" value="0.178" />
   <xacro:body wheel_radius="${wheel_radius}" />
   <xacro:wheel side="fl" wheel_radius="${wheel_radius}"
@@ -19,4 +20,5 @@
   <xacro:wheel side="rr" wheel_radius="${wheel_radius}"
     x="${-wheel_separation_x / 2}" y="${-wheel_separation_y / 2}" />
-  <xacro:sar_ros2_control mock="$(arg mock)" wheel_radius="${wheel_radius}" baud_rate="$(arg baud_rate)" device="$(arg device)" />
+  <xacro:rplidar x="0.0" y="0.0" z="0.03"/>
+  <xacro:sar_ros2_control mock="$(arg mock)" baud_rate="$(arg baud_rate)" device="$(arg device)" />
 </robot>

File: sar_description/urdf/wheel.urdf.xacro (robot description, xacro)
@@ -2,5 +2,5 @@
 <robot xmlns:xacro="http://wiki.ros.org/xacro">
   <xacro:macro name="wheel" params="side wheel_radius x y">
-    <xacro:property name="wheel_thickness" value="0.05" />
+    <xacro:property name="wheel_thickness" value="0.031" />
     <xacro:property name="wheel_mass" value="0.4" />
     <joint name="${side}_wheel_joint" type="continuous">

Commit message: Revert "Add rplidar to description"
This reverts commit e6d42fd9e6ba8fafbd727d230e154d898e937af2.

File: sar_description/urdf/body.urdf.xacro (robot description, xacro)
@@ -11,5 +11,5 @@
       <visual>
         <geometry>
-          <box size="0.240 0.178 0.060" />
+          <box size="0.240 0.220 0.060" />
         </geometry>
         <material name="dark_grey">
@@ -19,5 +19,5 @@
       <collision>
         <geometry>
-          <box size="0.240 0.178 0.060" />
+          <box size="0.240 0.220 0.060" />
         </geometry>
       </collision>

File: sar_description/urdf/ros2_control.urdf.xacro (robot description, xacro)
@@ -1,5 +1,5 @@
 <?xml version="1.0"?>
 <robot xmlns:xacro="http://wiki.ros.org/xacro">
-  <xacro:macro name="sar_ros2_control" params="mock:=false baud_rate:=115200 device:=/dev/ttyACM0">
+  <xacro:macro name="sar_ros2_control" params="mock:=false wheel_radius:=0.0 baud_rate:=115200 device:=/dev/ttyACM0">
     <ros2_control name="SarSystemHardware" type="system">
       <hardware>
@@ -8,19 +8,24 @@
         <param name="baud_rate">${baud_rate}</param>
         <param name="mock">${mock}</param>
+        <param name="wheel_radius">${wheel_radius}</param>
       </hardware>
       <joint name="fl_wheel_joint">
         <command_interface name="velocity" />
+        <state_interface name="position" />
         <state_interface name="velocity" />
       </joint>
       <joint name="fr_wheel_joint">
         <command_interface name="velocity" />
+        <state_interface name="position" />
         <state_interface name="velocity" />
       </joint>
       <joint name="rl_wheel_joint">
         <command_interface name="velocity" />
+        <state_interface name="position" />
         <state_interface name="velocity" />
       </joint>
       <joint name="rr_wheel_joint">
         <command_interface name="velocity" />
+        <state_interface name="position" />
         <state_interface name="velocity" />
       </joint>

File: sar_description/urdf/sar_robot.urdf.xacro (robot description, xacro)
@@ -7,8 +7,7 @@
   <xacro:include filename="$(find sar_description)/urdf/wheel.urdf.xacro" />
   <xacro:include filename="$(find sar_description)/urdf/ros2_control.urdf.xacro" />
-  <xacro:include filename="$(find sar_description)/urdf/rplidar.urdf.xacro" />
-  <xacro:property name="wheel_radius" value="0.03" />
-  <xacro:property name="wheel_separation_x" value="0.180" />
-  <xacro:property name="wheel_separation_y" value="0.178" />
+  <xacro:property name="wheel_radius" value="0.050" />
+  <xacro:property name="wheel_separation_x" value="0.170" />
+  <xacro:property name="wheel_separation_y" value="0.270" />
   <xacro:body wheel_radius="${wheel_radius}" />
   <xacro:wheel side="fl" wheel_radius="${wheel_radius}"
@@ -20,5 +19,4 @@
   <xacro:wheel side="rr" wheel_radius="${wheel_radius}"
     x="${-wheel_separation_x / 2}" y="${-wheel_separation_y / 2}" />
-  <xacro:rplidar x="0.0" y="0.0" z="0.03"/>
-  <xacro:sar_ros2_control mock="$(arg mock)" baud_rate="$(arg baud_rate)" device="$(arg device)" />
+  <xacro:sar_ros2_control mock="$(arg mock)" wheel_radius="${wheel_radius}" baud_rate="$(arg baud_rate)" device="$(arg device)" />
 </robot>

File: sar_description/urdf/wheel.urdf.xacro (robot description, xacro)
@@ -2,5 +2,5 @@
 <robot xmlns:xacro="http://wiki.ros.org/xacro">
   <xacro:macro name="wheel" params="side wheel_radius x y">
-    <xacro:property name="wheel_thickness" value="0.031" />
+    <xacro:property name="wheel_thickness" value="0.05" />
     <xacro:property name="wheel_mass" value="0.4" />
     <joint name="${side}_wheel_joint" type="continuous">

Commit message: Update with model & real robot measurements
Co-Authored-By: peter2395 <48293087+peter2395@users.noreply.github.com>

File: sar_description/urdf/body.urdf.xacro (robot description, xacro)
@@ -3,18 +3,23 @@
   <xacro:macro name="body" params="wheel_radius">
     <link name="base_link" />
+    <link name="base_footprint" />
+    <joint name="base_to_footprint" type="fixed">
+      <origin xyz="0 0 0" rpy="0.0 0.0 0.0" />1
+      <parent link="base_link" />
+      <child link="base_footprint" />
+    </joint>
     <joint name="base_to_body_joint" type="fixed">
-      <origin xyz="0.0 0.0 ${wheel_radius}" rpy="0.0 0.0 0.0" />
+      <origin xyz="0 0 ${wheel_radius}" rpy="0.0 0.0 0.0" />
       <parent link="base_link" />
       <child link="body_link" />
     </joint>
     <link name="body_link">
-      <visual>
-        <geometry>
-          <box size="0.240 0.178 0.060" />
-        </geometry>
-        <material name="dark_grey">
-          <color rgba="0.3 0.3 0.3 1.0" />
-        </material>
-      </visual>
+    <visual name="base_visual">
+      <origin xyz="0.115 -0.0875 0" rpy="0 0 0"/>
+      <geometry>
+        <mesh filename="package://sar_robot_description/meshes/SAR2.dae"
+              scale="0.001 0.001 0.001"/>
+      </geometry>
+    </visual>
       <collision>
         <geometry>

File: sar_description/urdf/rplidar.urdf.xacro (robot description, xacro)
@@ -4,13 +4,13 @@
     <joint name="rplidar_joint" type="fixed">
       <parent link="body_link" />
-      <child link="rplidar_link" />
+      <child link="laser_frame" />
       <origin xyz="${x} ${y} ${z}" rpy="0.0 0.0 0.0" />
     </joint>
-    <link name="rplidar_link">
+    <link name="laser_frame">
       <visual>
         <geometry>
-          <mesh filename="file://$(find sar_description)/meshes/rplidar_main.STL" scale="0.002 0.002 0.002" />
+          <mesh filename="package://sar_robot_description/meshes/RPLIDAR.dae" scale="0.001 0.001 0.001"/>
         </geometry>
-        <origin xyz="-0.07 0.067 0.0" rpy="${pi/2} 0.0 0.0" />
+        <origin xyz="-0.07 0.015 -0.036" rpy="0 0.0 ${pi}" />
         <material name="rplidar_color">
           <color rgba="0.1 0.1 0.1 1.0" />

File: sar_description/urdf/sar_robot.urdf.xacro (robot description, xacro)
@@ -7,7 +7,9 @@
   <xacro:include filename="$(find sar_description)/urdf/wheel.urdf.xacro" />
   <xacro:include filename="$(find sar_description)/urdf/ros2_control.urdf.xacro" />
+  <xacro:include filename="$(find sar_description)/urdf/rplidar.urdf.xacro" />
+  <xacro:include filename="$(find sar_description)/urdf/realsense.urdf.xacro" />
   <xacro:property name="wheel_radius" value="0.03" />
-  <xacro:property name="wheel_separation_x" value="0.180" />
-  <xacro:property name="wheel_separation_y" value="0.178" />
+  <xacro:property name="wheel_separation_x" value="0.200" />
+  <xacro:property name="wheel_separation_y" value="0.190" />
   <xacro:body wheel_radius="${wheel_radius}" />
   <xacro:wheel side="fl" wheel_radius="${wheel_radius}"
@@ -19,5 +21,6 @@
   <xacro:wheel side="rr" wheel_radius="${wheel_radius}"
     x="${-wheel_separation_x / 2}" y="${-wheel_separation_y / 2}" />
-  <!--<xacro:rplidar x="0.0" y="0.0" z="0.03"/>-->
+  <xacro:rplidar x="0.0" y="0.0" z="0.14" />
+  <xacro:realsense x="0.1375" y="0" z="0.0625" />
   <xacro:sar_ros2_control mock="$(arg mock)" baud_rate="$(arg baud_rate)" device="$(arg device)" />
 </robot>

File: sar_description/urdf/wheel.urdf.xacro (robot description, xacro)
@@ -14,8 +14,9 @@
     <link name="${side}_wheel_link">
       <visual>
-        <geometry>
-          <cylinder radius="${wheel_radius}" length="${wheel_thickness}" />
-        </geometry>
-        <origin xyz="0.0 0.0 0.0" rpy="${pi/2} 0.0 0.0" />
+      <geometry>
+        <mesh filename="package://sar_description/meshes/WHEEL.dae"
+              scale="0.0011 0.0011 0.0011"/>
+      </geometry>
+        <origin xyz="-0.07 -0.015 -0.022" rpy="0.0 0.0 ${pi/2}" />
         <material name="wheel_color">
           <color rgba="0.1 0.1 0.1 1.0" />

Commit message: Add inertial tags
Based on Invertor's values

File: sar_description/urdf/body.urdf.xacro (robot description, xacro)
@@ -29,7 +29,7 @@
       <inertial>
         <mass value="3.0" />
-        <inertia ixx="0.013" ixy="0.0" ixz="0.0"
-                              iyy="0.010" iyz="0.0"
-                                          izz="0.019" />
+        <inertia ixx="0.019480348" ixy="0.006659356" ixz="-0.010307569"
+                              iyy="0.040014748" iyz="0.004784591"
+                                          izz="0.028414280" />
       </inertial>
     </link>

File: sar_description/urdf/realsense.urdf.xacro (robot description, xacro)
@@ -21,4 +21,10 @@
       </geometry>
     </collision>
+    <inertial>
+		<mass value="0.048" />
+		<inertia ixx="0.000007287" ixy="0.000000001" ixz="-0.0"
+		                          iyy="0.000030308" iyz="0.000000021"
+		                                           izz="0.000033416" />
+	</inertial>
   </link>
   </xacro:macro>

File: sar_description/urdf/rplidar.urdf.xacro (robot description, xacro)
@@ -23,4 +23,10 @@
         <origin xyz="0.0 0.0 0.085" rpy="0.0 0.0 0.0" />
       </collision>
+	  <inertial>
+        <mass value="0.074" />
+        <inertia ixx="0.000083583" ixy="0.000110656" ixz="-0.000052990"
+                                  iyy="0.000323563" iyz="0.000021981"
+                                                   izz="0.000345389" />
+      </inertial>
     </link>
   </xacro:macro>

File: sar_description/urdf/wheel.urdf.xacro (robot description, xacro)
@@ -31,7 +31,7 @@
       <inertial>
         <mass value="${wheel_mass}" />
-        <inertia ixx="0.0003145" ixy="0.0" ixz="0.0"
-                                  iyy="0.0004561" iyz="0.0"
-                                                   izz="0.0003145" />
+        <inertia ixx="0.000228454" ixy="-0.000015215" ixz="-0.000043405"
+                                  iyy="0.000209819" iyz="-0.000066187"
+                                                   izz="0.000044202" />
       </inertial>
     </link>

Commit message: fix(sar_description): fix xacro parse error and mesh package URIs

File: sar_description/urdf/body.urdf.xacro (robot description, xacro)
@@ -5,5 +5,5 @@
     <link name="base_footprint" />
     <joint name="base_to_footprint" type="fixed">
-      <origin xyz="0 0 0" rpy="0.0 0.0 0.0" />1
+      <origin xyz="0 0 0" rpy="0.0 0.0 0.0" />
       <parent link="base_link" />
       <child link="base_footprint" />
@@ -18,5 +18,5 @@
       <origin xyz="0.115 -0.0875 0" rpy="0 0 0"/>
       <geometry>
-        <mesh filename="package://sar_robot_description/meshes/SAR2.dae"
+        <mesh filename="package://sar_description/meshes/SAR2.dae"
               scale="0.001 0.001 0.001"/>
       </geometry>

File: sar_description/urdf/realsense.urdf.xacro (robot description, xacro)
@@ -11,5 +11,5 @@
       <origin xyz="0 0 0" rpy="1.5708 0 0"/>
       <geometry>
-        <mesh filename="package://sar_robot_description/meshes/Realsense.dae"
+        <mesh filename="package://sar_description/meshes/Realsense.dae"
               scale="0.001 0.001 0.001"/>
       </geometry>

File: sar_description/urdf/rplidar.urdf.xacro (robot description, xacro)
@@ -10,5 +10,5 @@
       <visual>
         <geometry>
-          <mesh filename="package://sar_robot_description/meshes/RPLIDAR.dae" scale="0.001 0.001 0.001"/>
+          <mesh filename="package://sar_description/meshes/RPLIDAR.dae" scale="0.001 0.001 0.001"/>
         </geometry>
         <origin xyz="-0.07 0.015 -0.036" rpy="0 0.0 ${pi}" />
