Commit message: feat(sar_description): add camera optical frame for ROS image conventions
camera_frame is X-forward (REP-103 body convention), but OpenCV/PnP and
the gz camera sensor produce pixel data in the optical convention
(Z-forward, X-right, Y-down). Add a child camera_optical_frame rotated
by (-pi/2, 0, -pi/2) and tag the gz sensor's images with it, so
downstream consumers (e.g. sar_perception) can do TF lookups on the
image's frame_id and get the right transform without any in-node hacks.

File: sar_description/urdf/gazebo.urdf.xacro (robot description, xacro)
@@ -50,5 +50,5 @@
         <always_on>true</always_on>
         <visualize>false</visualize>
-        <gz_frame_id>camera_frame</gz_frame_id>
+        <gz_frame_id>camera_optical_frame</gz_frame_id>
         <camera>
           <horizontal_fov>1.211</horizontal_fov>

File: sar_description/urdf/sensors/realsense.urdf.xacro (robot description, xacro)
@@ -28,4 +28,10 @@
 	</inertial>
   </link>
+  <joint name="camera_optical_joint" type="fixed">
+    <parent link="camera_frame"/>
+    <child link="camera_optical_frame"/>
+    <origin xyz="0 0 0" rpy="-1.5708 0 -1.5708"/>
+  </joint>
+  <link name="camera_optical_frame"/>
   </xacro:macro>
 </robot>
