Commit message: feat(sar_description): add gazebo sim support with mecanum friction
Introduce a use_sim xacro arg that gates Gazebo-only content so the
same URDF drives both the real robot and gz-sim.

- gazebo.urdf.xacro: gz_ros2_control-system plugin plus gpu_lidar,
  camera, and imu sensor tags on existing frames.
- ros2_control: switch hardware plugin between sar_control/SarSystem
  (real) and gz_ros2_control/GazeboSimSystem (sim); add position state
  interfaces in sim for odometry.
- wheel: in sim, swap visual for rosbot_description mecanum_{a,b}.dae
  scaled to our wheel_radius, and emit an anisotropic-friction gazebo
  block (mu/mu2/slip/fdir1 expressed_in=base_link) matching Husarion's
  tuned values per corner.
- description.launch.py: forward use_sim to xacro and apply
  use_sim_time on robot_state_publisher.
- package.xml: depend on rosbot_description for mecanum meshes.

File: sar_description/urdf/base/wheel.urdf.xacro (robot description, xacro)
@@ -1,7 +1,8 @@
 <?xml version="1.0"?>
 <robot xmlns:xacro="http://wiki.ros.org/xacro">
-  <xacro:macro name="wheel" params="side wheel_radius x y">
+  <xacro:macro name="wheel" params="side wheel_radius x y use_sim:=false variant:=a fdir:='1 1 0'">
     <xacro:property name="wheel_thickness" value="0.031" />
     <xacro:property name="wheel_mass" value="0.4" />
+    <xacro:property name="mecanum_mesh_scale" value="${wheel_radius / 0.05}" />
     <joint name="${side}_wheel_joint" type="continuous">
       <parent link="body_link" />
@@ -14,12 +15,21 @@
     <link name="${side}_wheel_link">
       <visual>
-      <geometry>
-        <mesh filename="package://sar_description/meshes/wheel.dae"
-              scale="0.0011 0.0011 0.0011"/>
-      </geometry>
-        <origin xyz="-0.07 -0.015 -0.022" rpy="0.0 0.0 ${pi/2}" />
-        <material name="wheel_color">
-          <color rgba="0.1 0.1 0.1 1.0" />
-        </material>
+        <xacro:if value="${use_sim}">
+          <geometry>
+            <mesh filename="package://rosbot_description/meshes/rosbot_xl/mecanum_${variant}.dae"
+                  scale="${mecanum_mesh_scale} ${mecanum_mesh_scale} ${mecanum_mesh_scale}"/>
+          </geometry>
+          <origin xyz="0.0 0.0 0.0" rpy="0.0 0.0 0.0" />
+        </xacro:if>
+        <xacro:unless value="${use_sim}">
+          <geometry>
+            <mesh filename="package://sar_description/meshes/wheel.dae"
+                  scale="0.0011 0.0011 0.0011"/>
+          </geometry>
+          <origin xyz="-0.07 -0.015 -0.022" rpy="0.0 0.0 ${pi/2}" />
+          <material name="wheel_color">
+            <color rgba="0.1 0.1 0.1 1.0" />
+          </material>
+        </xacro:unless>
       </visual>
       <collision>
@@ -36,4 +46,21 @@
       </inertial>
     </link>
+    <xacro:if value="${use_sim}">
+      <gazebo reference="${side}_wheel_link" xmlns:ignition="http://ignitionrobotics.org/schema">
+        <collision>
+          <surface>
+            <friction>
+              <ode>
+                <mu>0.8</mu>
+                <mu2>0.2</mu2>
+                <slip1>0.035</slip1>
+                <slip2>0</slip2>
+                <fdir1 ignition:expressed_in="base_link">${fdir}</fdir1>
+              </ode>
+            </friction>
+          </surface>
+        </collision>
+      </gazebo>
+    </xacro:if>
   </xacro:macro>
 </robot>

File: sar_description/urdf/control/ros2_control.urdf.xacro (robot description, xacro)
@@ -1,27 +1,44 @@
 <?xml version="1.0"?>
 <robot xmlns:xacro="http://wiki.ros.org/xacro">
-  <xacro:macro name="sar_ros2_control" params="mock:=false baud_rate:=115200 device:=/dev/ttyACM0">
+  <xacro:macro name="sar_ros2_control" params="use_sim:=false mock:=false baud_rate:=115200 device:=/dev/ttyACM0">
     <ros2_control name="sar_system" type="system">
       <hardware>
-        <plugin>sar_control/SarSystemHardware</plugin>
-        <param name="device">${device}</param>
-        <param name="baud_rate">${baud_rate}</param>
-        <param name="mock">${mock}</param>
+        <xacro:if value="${use_sim}">
+          <plugin>gz_ros2_control/GazeboSimSystem</plugin>
+        </xacro:if>
+        <xacro:unless value="${use_sim}">
+          <plugin>sar_control/SarSystemHardware</plugin>
+          <param name="device">${device}</param>
+          <param name="baud_rate">${baud_rate}</param>
+          <param name="mock">${mock}</param>
+        </xacro:unless>
       </hardware>
       <joint name="fl_wheel_joint">
         <command_interface name="velocity" />
         <state_interface name="velocity" />
+        <xacro:if value="${use_sim}">
+          <state_interface name="position" />
+        </xacro:if>
       </joint>
       <joint name="fr_wheel_joint">
         <command_interface name="velocity" />
         <state_interface name="velocity" />
+        <xacro:if value="${use_sim}">
+          <state_interface name="position" />
+        </xacro:if>
       </joint>
       <joint name="rl_wheel_joint">
         <command_interface name="velocity" />
         <state_interface name="velocity" />
+        <xacro:if value="${use_sim}">
+          <state_interface name="position" />
+        </xacro:if>
       </joint>
       <joint name="rr_wheel_joint">
         <command_interface name="velocity" />
         <state_interface name="velocity" />
+        <xacro:if value="${use_sim}">
+          <state_interface name="position" />
+        </xacro:if>
       </joint>
     </ros2_control>

File: sar_description/urdf/sar_robot.urdf.xacro (robot description, xacro)
@@ -1,7 +1,11 @@
 <?xml version="1.0"?>
 <robot name="sar_robot" xmlns:xacro="http://wiki.ros.org/xacro">
+  <xacro:arg name="use_sim" default="false" />
   <xacro:arg name="mock" default="false" />
   <xacro:arg name="baud_rate" default="115200" />
   <xacro:arg name="device" default="/dev/ttyACM0" />
+  <xacro:arg name="namespace" default="" />
+  <xacro:arg name="controllers_config"
+             default="$(find sar_control)/config/controllers.yaml" />
   <xacro:include filename="$(find sar_description)/urdf/base/body.urdf.xacro" />
   <xacro:include filename="$(find sar_description)/urdf/base/wheel.urdf.xacro" />
@@ -14,13 +18,23 @@
   <xacro:body wheel_radius="${wheel_radius}" />
   <xacro:wheel side="fl" wheel_radius="${wheel_radius}"
-    x="${wheel_separation_x / 2}" y="${wheel_separation_y / 2}" />
+    x="${wheel_separation_x / 2}" y="${wheel_separation_y / 2}"
+    use_sim="$(arg use_sim)" variant="b" fdir="1 -1 0" />
   <xacro:wheel side="fr" wheel_radius="${wheel_radius}"
-    x="${wheel_separation_x / 2}" y="${-wheel_separation_y / 2}" />
+    x="${wheel_separation_x / 2}" y="${-wheel_separation_y / 2}"
+    use_sim="$(arg use_sim)" variant="a" fdir="1 1 0" />
   <xacro:wheel side="rl" wheel_radius="${wheel_radius}"
-    x="${-wheel_separation_x / 2}" y="${wheel_separation_y / 2}" />
+    x="${-wheel_separation_x / 2}" y="${wheel_separation_y / 2}"
+    use_sim="$(arg use_sim)" variant="a" fdir="1 1 0" />
   <xacro:wheel side="rr" wheel_radius="${wheel_radius}"
-    x="${-wheel_separation_x / 2}" y="${-wheel_separation_y / 2}" />
+    x="${-wheel_separation_x / 2}" y="${-wheel_separation_y / 2}"
+    use_sim="$(arg use_sim)" variant="b" fdir="1 -1 0" />
   <xacro:rplidar x="0.0" y="0.0" z="0.14" />
   <xacro:realsense x="0.1375" y="0" z="0.0625" />
-  <xacro:sar_ros2_control mock="$(arg mock)" baud_rate="$(arg baud_rate)" device="$(arg device)" />
+  <xacro:sar_ros2_control use_sim="$(arg use_sim)" mock="$(arg mock)"
+    baud_rate="$(arg baud_rate)" device="$(arg device)" />
+  <xacro:if value="$(arg use_sim)">
+    <xacro:include filename="$(find sar_description)/urdf/gazebo.urdf.xacro" />
+    <xacro:sar_gazebo controllers_config="$(arg controllers_config)"
+      namespace="$(arg namespace)" />
+  </xacro:if>
 </robot>
