Commit message: refactor(sar_description): normalize mesh filenames and update URDF references

File: sar_description/urdf/base/body.urdf.xacro (robot description, xacro)
@@ -18,5 +18,5 @@
       <origin xyz="0.115 -0.0875 0" rpy="0 0 0"/>
       <geometry>
-        <mesh filename="package://sar_description/meshes/SAR2.dae"
+        <mesh filename="package://sar_description/meshes/sar_body.dae"
               scale="0.001 0.001 0.001"/>
       </geometry>

File: sar_description/urdf/base/wheel.urdf.xacro (robot description, xacro)
@@ -15,5 +15,5 @@
       <visual>
       <geometry>
-        <mesh filename="package://sar_description/meshes/WHEEL.dae"
+        <mesh filename="package://sar_description/meshes/wheel.dae"
               scale="0.0011 0.0011 0.0011"/>
       </geometry>

File: sar_description/urdf/sensors/realsense.urdf.xacro (robot description, xacro)
@@ -11,5 +11,5 @@
       <origin xyz="0 0 0" rpy="1.5708 0 0"/>
       <geometry>
-        <mesh filename="package://sar_description/meshes/Realsense.dae"
+        <mesh filename="package://sar_description/meshes/realsense.dae"
               scale="0.001 0.001 0.001"/>
       </geometry>

File: sar_description/urdf/sensors/rplidar.urdf.xacro (robot description, xacro)
@@ -10,5 +10,5 @@
       <visual>
         <geometry>
-          <mesh filename="package://sar_description/meshes/RPLIDAR.dae" scale="0.001 0.001 0.001"/>
+          <mesh filename="package://sar_description/meshes/rplidar.dae" scale="0.001 0.001 0.001"/>
         </geometry>
         <origin xyz="-0.07 0.015 -0.036" rpy="0 0.0 ${pi}" />

Commit message: fix(sar): switch to ign_ros2_control and match ROSbot XL physics
The gz_ros2_control-system plugin on Gazebo Fortress (Sim 6) did not
deliver unstamped Twist messages to the controller under this setup,
and the SAR scale (30 mm wheels, 3 kg body) was below the friction
threshold needed for mecanum rotation. Both issues are resolved by
aligning with Husarion's working ROSbot XL configuration.

- sar_description/urdf/gazebo.urdf.xacro: use the Fortress-native
  ign_ros2_control-system plugin and ign_ros2_control::IgnitionROS2ControlPlugin.
- sar_description/urdf/control/ros2_control.urdf.xacro: switch sim
  hardware plugin to ign_ros2_control/IgnitionSystem.
- sar_description/urdf/sar_robot.urdf.xacro: adopt ROSbot XL
  dimensions (wheel_radius=0.05, wheel_separation_x=0.170,
  wheel_separation_y=0.270).
- sar_description/urdf/base/wheel.urdf.xacro: wheel thickness 0.05 and
  principal-axis inertia; Husarion-tuned anisotropic friction
  (mu=0.8, mu2=0.2, slip1=0.035).
- sar_description/urdf/base/body.urdf.xacro: body mass 3.5 kg with
  zeroed off-diagonal inertia matching ROSbot XL.
- sar_control/config/controllers.yaml: full Husarion mecanum config
  with use_stamped_vel=false, velocity/acceleration limits, and
  wheel separation/radius multipliers.
- sar_gazebo/config/gz_bridge.yaml: bridge gz /cmd_vel (gz.msgs.Twist)
  to ROS /cmd_vel so the gz GUI Teleop reaches the controller.
- sar_gazebo/launch/gazebo.launch.py: default husarion_world spawn
  moved to (0, -2.5, 0.2) to clear the wall at the origin.

File: sar_description/urdf/base/body.urdf.xacro (robot description, xacro)
@@ -28,8 +28,8 @@
       </collision>
       <inertial>
-        <mass value="3.0" />
-        <inertia ixx="0.019480348" ixy="0.006659356" ixz="-0.010307569"
-                              iyy="0.040014748" iyz="0.004784591"
-                                          izz="0.028414280" />
+        <mass value="3.5" />
+        <inertia ixx="0.01393" ixy="0.0" ixz="0.0"
+                               iyy="0.01081" iyz="0.0"
+                                             izz="0.02048" />
       </inertial>
     </link>

File: sar_description/urdf/base/wheel.urdf.xacro (robot description, xacro)
@@ -2,5 +2,5 @@
 <robot xmlns:xacro="http://wiki.ros.org/xacro">
   <xacro:macro name="wheel" params="side wheel_radius x y use_sim:=false variant:=a fdir:='1 1 0'">
-    <xacro:property name="wheel_thickness" value="0.031" />
+    <xacro:property name="wheel_thickness" value="0.05" />
     <xacro:property name="wheel_mass" value="0.4" />
     <xacro:property name="mecanum_mesh_scale" value="${wheel_radius / 0.05}" />
@@ -41,7 +41,7 @@
       <inertial>
         <mass value="${wheel_mass}" />
-        <inertia ixx="0.000228454" ixy="-0.000015215" ixz="-0.000043405"
-                                  iyy="0.000209819" iyz="-0.000066187"
-                                                   izz="0.000044202" />
+        <inertia ixx="0.0003145" ixy="0.0" ixz="0.0"
+                                 iyy="0.0004561" iyz="0.0"
+                                                 izz="0.0003145" />
       </inertial>
     </link>

File: sar_description/urdf/control/ros2_control.urdf.xacro (robot description, xacro)
@@ -5,5 +5,5 @@
       <hardware>
         <xacro:if value="${use_sim}">
-          <plugin>gz_ros2_control/GazeboSimSystem</plugin>
+          <plugin>ign_ros2_control/IgnitionSystem</plugin>
         </xacro:if>
         <xacro:unless value="${use_sim}">

File: sar_description/urdf/gazebo.urdf.xacro (robot description, xacro)
@@ -3,6 +3,6 @@
   <xacro:macro name="sar_gazebo" params="controllers_config namespace:=''">
     <gazebo>
-      <plugin filename="gz_ros2_control-system"
-              name="gz_ros2_control::GazeboSimROS2ControlPlugin">
+      <plugin filename="ign_ros2_control-system"
+              name="ign_ros2_control::IgnitionROS2ControlPlugin">
         <parameters>${controllers_config}</parameters>
         <ros>
@@ -10,4 +10,6 @@
             <namespace>${namespace}</namespace>
           </xacro:if>
+          <remapping>mecanum_drive_controller/cmd_vel_unstamped:=cmd_vel</remapping>
+          <remapping>mecanum_drive_controller/odom:=odometry/wheels</remapping>
         </ros>
       </plugin>

File: sar_description/urdf/sar_robot.urdf.xacro (robot description, xacro)
@@ -13,7 +13,7 @@
   <xacro:include filename="$(find sar_description)/urdf/sensors/rplidar.urdf.xacro" />
   <xacro:include filename="$(find sar_description)/urdf/sensors/realsense.urdf.xacro" />
-  <xacro:property name="wheel_radius" value="0.03" />
-  <xacro:property name="wheel_separation_x" value="0.200" />
-  <xacro:property name="wheel_separation_y" value="0.190" />
+  <xacro:property name="wheel_radius" value="0.05" />
+  <xacro:property name="wheel_separation_x" value="0.170" />
+  <xacro:property name="wheel_separation_y" value="0.270" />
   <xacro:body wheel_radius="${wheel_radius}" />
   <xacro:wheel side="fl" wheel_radius="${wheel_radius}"

Commit message: feat(sar): split sim and real physics via use_sim
ODE cannot reliably simulate mecanum wheels at SAR's real 30 mm scale
(rotation torque arm is too small; wheels stick in place). Solve it by
decoupling sim physics from real kinematics: sim runs with ROSbot XL
scale parameters that are known to work, the real robot keeps its true
dimensions for the hardware controller.

- sar_description/urdf/sar_robot.urdf.xacro: select wheel_radius (0.05
  sim / 0.03 real), wheel_separation_x (0.170 / 0.200), and
  wheel_separation_y (0.270 / 0.190) based on the use_sim arg.
- sar_description/urdf/base/body.urdf.xacro: use ROSbot XL body mass
  and diagonal inertia in sim, the original CAD mass/tensor on the real
  robot.
- sar_description/urdf/base/wheel.urdf.xacro: wheel thickness 0.05 sim
  / 0.031 real, with matching inertia tensors.
- sar_control/config/controllers.yaml: restore real-robot kinematics
  (30 mm wheels, 0.200x0.190 stance, multipliers at 1.0). These were
  temporarily overridden during sim debugging.
- sar_control/config/controllers_sim.yaml: new sim-only config that
  matches the sim URDF (50 mm wheels, 0.170x0.270 stance, Husarion's
  0.95 correction multipliers) and raises velocity/acceleration limits
  for responsive teleop.

File: sar_description/urdf/base/body.urdf.xacro (robot description, xacro)
@@ -27,10 +27,20 @@
         </geometry>
       </collision>
-      <inertial>
-        <mass value="3.5" />
-        <inertia ixx="0.01393" ixy="0.0" ixz="0.0"
-                               iyy="0.01081" iyz="0.0"
-                                             izz="0.02048" />
-      </inertial>
+      <xacro:if value="$(arg use_sim)">
+        <inertial>
+          <mass value="3.5" />
+          <inertia ixx="0.01393" ixy="0.0" ixz="0.0"
+                                 iyy="0.01081" iyz="0.0"
+                                               izz="0.02048" />
+        </inertial>
+      </xacro:if>
+      <xacro:unless value="$(arg use_sim)">
+        <inertial>
+          <mass value="3.0" />
+          <inertia ixx="0.019480348" ixy="0.006659356" ixz="-0.010307569"
+                                iyy="0.040014748" iyz="0.004784591"
+                                            izz="0.028414280" />
+        </inertial>
+      </xacro:unless>
     </link>
     <joint name="body_to_imu_joint" type="fixed">

File: sar_description/urdf/base/wheel.urdf.xacro (robot description, xacro)
@@ -2,5 +2,10 @@
 <robot xmlns:xacro="http://wiki.ros.org/xacro">
   <xacro:macro name="wheel" params="side wheel_radius x y use_sim:=false variant:=a fdir:='1 1 0'">
-    <xacro:property name="wheel_thickness" value="0.05" />
+    <xacro:if value="${use_sim}">
+      <xacro:property name="wheel_thickness" value="0.05" />
+    </xacro:if>
+    <xacro:unless value="${use_sim}">
+      <xacro:property name="wheel_thickness" value="0.031" />
+    </xacro:unless>
     <xacro:property name="wheel_mass" value="0.4" />
     <xacro:property name="mecanum_mesh_scale" value="${wheel_radius / 0.05}" />
@@ -41,7 +46,14 @@
       <inertial>
         <mass value="${wheel_mass}" />
-        <inertia ixx="0.0003145" ixy="0.0" ixz="0.0"
-                                 iyy="0.0004561" iyz="0.0"
-                                                 izz="0.0003145" />
+        <xacro:if value="${use_sim}">
+          <inertia ixx="0.0003145" ixy="0.0" ixz="0.0"
+                                   iyy="0.0004561" iyz="0.0"
+                                                   izz="0.0003145" />
+        </xacro:if>
+        <xacro:unless value="${use_sim}">
+          <inertia ixx="0.000228454" ixy="-0.000015215" ixz="-0.000043405"
+                                    iyy="0.000209819" iyz="-0.000066187"
+                                                     izz="0.000044202" />
+        </xacro:unless>
       </inertial>
     </link>

File: sar_description/urdf/sar_robot.urdf.xacro (robot description, xacro)
@@ -13,7 +13,14 @@
   <xacro:include filename="$(find sar_description)/urdf/sensors/rplidar.urdf.xacro" />
   <xacro:include filename="$(find sar_description)/urdf/sensors/realsense.urdf.xacro" />
-  <xacro:property name="wheel_radius" value="0.05" />
-  <xacro:property name="wheel_separation_x" value="0.170" />
-  <xacro:property name="wheel_separation_y" value="0.270" />
+  <xacro:if value="$(arg use_sim)">
+    <xacro:property name="wheel_radius" value="0.05" />
+    <xacro:property name="wheel_separation_x" value="0.170" />
+    <xacro:property name="wheel_separation_y" value="0.270" />
+  </xacro:if>
+  <xacro:unless value="$(arg use_sim)">
+    <xacro:property name="wheel_radius" value="0.03" />
+    <xacro:property name="wheel_separation_x" value="0.200" />
+    <xacro:property name="wheel_separation_y" value="0.190" />
+  </xacro:unless>
   <xacro:body wheel_radius="${wheel_radius}" />
   <xacro:wheel side="fl" wheel_radius="${wheel_radius}"
