Commit message: fix(sar_description): point realsense camera forward in sim
The realsense joint had a 90 deg yaw, which made the gz camera sensor
look sideways into the robot housing instead of along +X. Zero the joint
rotation and compose the same world-frame mesh orientation in the visual.

File: sar_description/urdf/sensors/realsense.urdf.xacro (robot description, xacro)
@@ -5,9 +5,9 @@
     <parent link="body_link"/>
     <child link="camera_frame"/>
-    <origin xyz="${x} ${y} ${z}" rpy="0 0 1.5708"/>
+    <origin xyz="${x} ${y} ${z}" rpy="0 0 0"/>
   </joint>
   <link name="camera_frame">
     <visual>
-      <origin xyz="0 0 0" rpy="1.5708 0 0"/>
+      <origin xyz="0 0 0" rpy="1.5708 0 1.5708"/>
       <geometry>
         <mesh filename="package://sar_description/meshes/realsense.dae"
